File: pcb/aalborg_mfc_interface.sch (KiCad schematic (older format))
At the start: 4 parts

Commit message: Added some schematic components.
Parts:
- removed J?: DB15, symbol DB15
- added C1, C2, C3: 10uF, symbol C
- added C4: 0.1uF, symbol C
- added D1: LED, symbol LED
- added E1: ENCODER_C14, symbol ENCODER_C14
- added P2: DISPLAY, symbol CONN_01X03
- added R1: 1.96k, symbol R
- added R2, R3: 5.1k, symbol R
- added REG1: CONV_DC_DC, symbol CONV_DC_DC
- added U1: MAX6817, symbol MAX6817
- J1: renamed from J?; value DB15 -> MFCA
- gave numbers to parts that had none: 2
Connections:
- net labels added: ANALOG_IN_A, ANALOG_OUT_A, D_ENC_BTN, ENC_A, ENC_B, ENC_BTN, PURGE_A, PURGE_B, TX3, VALVE_OFF_A, VALVE_OFF_B, V_IN
- net labels removed: CS, IN, MISO, MOSI, RST, SCK
- wire segments 22 -> 78
- no-connect marks 76 -> 81

Commit message: Initial board layout.
Parts:
- removed R1: 1.96k, symbol R
- added C5, C6: 10uF, symbol C
- added J2: MFCB, symbol DB15
- added R4, R5: 5.1k, symbol R
- renumbered R2 to R1, R3 to R2
Connections:
- net labels added: ANALOG_IN_B, ANALOG_OUT_B, PWM_A, PWM_B
- wire segments 78 -> 102
- no-connect marks 81 -> 83

Commit message: Initial pcb layout.
Parts:
- REG1: value CONV_DC_DC -> +12VDC
Changed lines of the file:
@@
 P 6800 850
 F 0 "REG1" H 7000 550 60  0000 C CNN
-F 1 "CONV_DC_DC" H 6800 950 60  0000 C CNN
+F 1 "+12VDC" H 6800 950 60  0000 C CNN
 F 2 "" H 6800 850 60  0000 C CNN
 F 3 "" H 6800 850 60  0000 C CNN
@@
 Wire Wire Line
 	850  6550 850  6750
+Text Label 1750 1850 0    60   ~ 0
+GND
 $EndSCHEMATC

Commit message: Initial version 1.1 design.
Parts:
- removed C1, C2, C3, C5, C6: 10uF, symbol C
- removed C4: 0.1uF, symbol C
- removed D1: LED, symbol LED
- removed J1: MFCA, symbol DB15
- removed J2: MFCB, symbol DB15
- removed P1: +24VDC, symbol CONN_01X02
- removed P2: DISPLAY, symbol CONN_01X03
- removed R1, R2, R4, R5: 5.1k, symbol R
- removed REG1: +12VDC, symbol CONV_DC_DC
- removed SHIELD1: ARDUINO_MEGA_SHIELD_FULL, symbol ARDUINO_MEGA_SHIELD_FULL
- added ARDUINO1: ARDUINO_MEGA, aalborg_mfc_interface:ARDUINO_MEGA_SHIELD, symbol ARDUINO_MEGA
- added C1, C2, C3, C5, C6: 10uF, aalborg_mfc_interface:SM1210, symbol 10uF
- added C4: 0.1uF, aalborg_mfc_interface:SM1210, symbol 0.1uF
- added D1: LED_24V, aalborg_mfc_interface:LED_555-3XXX, symbol LED_24V
- added J1, J2: DB15FV, aalborg_mfc_interface:DB15FD, symbol DB15FV
- added P1: PWR_JACK_2.5x5.5, aalborg_mfc_interface:DCJACK_2PIN_HIGHCURRENT, symbol PWR_JACK_2.5x5.5
- added P2: HEADER_01X03, aalborg_mfc_interface:Header_Shrouded_3_Pin, symbol HEADER_01X03
- added R1, R2, R3, R4: 5.11k, aalborg_mfc_interface:SM1210, symbol 5.11k
- added REG1: CONV_DC_DC_12V_1A, aalborg_mfc_interface:DC_DC_CONV_R78C, symbol CONV_DC_DC_12V_1A
- E1: footprint (none) -> aalborg_mfc_interface:Micro-MaTch_6_SMD; Description (none) -> ENCODER OPT 32PPR DET CABLE TYPE; PartNumber (none) -> 102-1914-ND; Vendor (none) -> digikey
- U1: footprint (none) -> aalborg_mfc_interface:MAX6817; Description (none) -> IC_DEBOUNCER_SWITCH_DUAL_SOT23-6; PartNumber (none) -> MAX6817EUT+TCT-ND; Vendor (none) -> digikey

Commit message: Cleaned up component descriptions.
Parts:
- ARDUINO1: Description BOARD_MCU_MEGA2560 -> BOARD MCU MEGA2560
- P2: Description BERGSTIK II .100\" SR STRAIGHT -> 01x03 .100 SR STRAIGHT
- REG1: Description CONV_DC/DC_1A_12V_OUT_SIP_VERT -> CONV DC/DC 1A 12V OUT SIP VERT
- U1: Description IC_DEBOUNCER_SWITCH_DUAL_SOT23-6 -> IC DEBOUNCER SWITCH DUAL SOT23-6
Changed lines of the file:
@@
 LIBS:valves
 LIBS:aalborg_mfc_interface
+LIBS:components
 LIBS:aalborg_mfc_interface-cache
 EELAYER 25 0
@@
 GND
 $Comp
-L MAX6817 U1
-U 1 1 5488E1D0
-P 4850 6950
-F 0 "U1" H 5100 6700 60  0000 C CNN
-F 1 "MAX6817" H 4850 7550 60  0000 C CNN
-F 2 "aalborg_mfc_interface:MAX6817" H 5000 6600 60  0001 C CNN
-F 3 "" H 4850 6950 60  0000 C CNN
-F 4 "digikey" H 5200 6800 60  0001 C CNN "Vendor"
-F 5 "MAX6817EUT+TCT-ND" H 5300 6900 60  0001 C CNN "PartNumber"
-F 6 "IC_DEBOUNCER_SWITCH_DUAL_SOT23-6" H 5400 7000 60  0001 C CNN "Description"
-	1    4850 6950
-	1    0    0    -1
-$EndComp
-$Comp
-L ARDUINO_MEGA ARDUINO1
-U 1 1 5488E846
-P 3250 3500
-F 0 "ARDUINO1" H 3300 6250 60  0000 C CNN
-F 1 "ARDUINO_MEGA" H 3250 800 60  0000 C CNN
-F 2 "aalborg_mfc_interface:ARDUINO_MEGA_SHIELD" H 3200 6150 60  0001 C CNN
-F 3 "" H 3300 6250 60  0000 C CNN
-F 4 "digikey" H 3400 6350 60  0001 C CNN "Vendor"
-F 5 "1050-1018-ND" H 3500 6450 60  0001 C CNN "PartNumber"
-F 6 "BOARD_MCU_MEGA2560" H 3600 6550 60  0001 C CNN "Description"
-	1    3250 3500
-	1    0    0    -1
-$EndComp
-$Comp
-L CONV_DC_DC_12V_1A REG1
-U 1 1 5488ECA7
-P 6800 850
-F 0 "REG1" H 7000 550 60  0000 C CNN
-F 1 "CONV_DC_DC_12V_1A" H 6800 950 60  0000 C CNN
-F 2 "aalborg_mfc_interface:DC_DC_CONV_R78C" H 6900 450 60  0001 C CNN
-F 3 "" H 6800 850 60  0000 C CNN
-F 4 "digikey" H 6800 650 60  0001 C CNN "Vendor"
-F 5 "945-1392-5-ND" H 6800 750 60  0001 C CNN "PartNumber"
-F 6 "CONV_DC/DC_1A_12V_OUT_SIP_VERT" H 7300 850 60  0001 C CNN "Description"
-	1    6800 850
-	1    0    0    -1
-$EndComp
-$Comp
 L ENCODER_C14 E1
 U 1 1 5488F1C1
@@
 	1    5700 1000
 	1    0    0    -1
-$EndComp
-$Comp
-L HEADER_01X03 P2
-U 1 1 548904D3
-P 6450 6150
-F 0 "P2" H 6450 6350 50  0000 C CNN
-F 1 "HEADER_01X03" V 6550 6150 50  0000 C CNN
-F 2 "aalborg_mfc_interface:Header_Shrouded_3_Pin" H 6350 6250 60  0001 C CNN
-F 3 "" H 6450 6150 60  0000 C CNN
-F 4 "digikey" H 6550 6450 60  0001 C CNN "Vendor"
-F 5 "609-3461-ND" H 6650 6550 60  0001 C CNN "PartNumber"
-F 6 "BERGSTIK II .100\" SR STRAIGHT" H 6750 6650 60  0001 C CNN "Description"
-	1    6450 6150
-	-1   0    0    1
 $EndComp
 $Comp
@@
 	0    1    1    0
 $EndComp
+$Comp
+L ARDUINO_MEGA ARDUINO1
+U 1 1 5489C516
+P 3250 3500
+F 0 "ARDUINO1" H 3300 6250 60  0000 C CNN
+F 1 "ARDUINO_MEGA" H 3250 800 60  0000 C CNN
+F 2 "aalborg_mfc_interface:ARDUINO_MEGA_SHIELD" H 3200 6150 60  0001 C CNN
+F 3 "" H 3300 6250 60  0000 C CNN
+F 4 "digikey" H 3400 6350 60  0001 C CNN "Vendor"
+F 5 "1050-1018-ND" H 3500 6450 60  0001 C CNN "PartNumber"
+F 6 "BOARD MCU MEGA2560" H 3600 6550 60  0001 C CNN "Description"
+	1    3250 3500
+	1    0    0    -1
+$EndComp
+$Comp
+L CONV_DC_DC_12V_1A REG1
+U 1 1 5489CB72
+P 6800 850
+F 0 "REG1" H 7000 550 60  0000 C CNN
+F 1 "CONV_DC_DC_12V_1A" H 6800 950 60  0000 C CNN
+F 2 "aalborg_mfc_interface:DC_DC_CONV_R78C" H 6900 450 60  0001 C CNN
+F 3 "" H 6800 850 60  0000 C CNN
+F 4 "digikey" H 6800 650 60  0001 C CNN "Vendor"
+F 5 "945-1392-5-ND" H 6800 750 60  0001 C CNN "PartNumber"
+F 6 "CONV DC/DC 1A 12V OUT SIP VERT" H 7300 850 60  0001 C CNN "Description"
+	1    6800 850
+	1    0    0    -1
+$EndComp
+$Comp
+L HEADER_01X03 P2
+U 1 1 5489D3E6
+P 6450 6150
+F 0 "P2" H 6450 6350 50  0000 C CNN
+F 1 "HEADER_01X03" V 6550 6150 50  0000 C CNN
+F 2 "aalborg_mfc_interface:Header_Shrouded_3_Pin" H 6350 6250 60  0001 C CNN
+F 3 "" H 6450 6150 60  0000 C CNN
+F 4 "digikey" H 6550 6450 60  0001 C CNN "Vendor"
+F 5 "609-3461-ND" H 6650 6550 60  0001 C CNN "PartNumber"
+F 6 "01x03 .100 SR STRAIGHT" H 6750 6650 60  0001 C CNN "Description"
+	1    6450 6150
+	-1   0    0    1
+$EndComp
+$Comp
+L MAX6817 U1
+U 1 1 5489DAE1
+P 4850 6950
+F 0 "U1" H 5100 6700 60  0000 C CNN
+F 1 "MAX6817" H 4850 7550 60  0000 C CNN
+F 2 "aalborg_mfc_interface:MAX6817" H 5000 6600 60  0001 C CNN
+F 3 "" H 4850 6950 60  0000 C CNN
+F 4 "digikey" H 5200 6800 60  0001 C CNN "Vendor"
+F 5 "MAX6817EUT+TCT-ND" H 5300 6900 60  0001 C CNN "PartNumber"
+F 6 "IC DEBOUNCER SWITCH DUAL SOT23-6" H 5400 7000 60  0001 C CNN "Description"
+	1    4850 6950
+	1    0    0    -1
+$EndComp
 $EndSCHEMATC

Commit message: Updated ENCODER_C14.
Parts:
- E1: Description ENCODER OPT 32PPR DET CABLE TYPE -> CONN FMALE-ON-BRD 6POS VERT SMD; PartNumber 102-1914-ND -> A99474CT-ND
Changed lines of the file:
@@
 GND
-$Comp
-L ENCODER_C14 E1
-U 1 1 5488F1C1
-P 1550 6950
-F 0 "E1" H 1550 6600 60  0000 C CNN
-F 1 "ENCODER_C14" H 1550 7300 60  0000 C CNN
-F 2 "aalborg_mfc_interface:Micro-MaTch_6_SMD" H 1450 6500 60  0001 C CNN
-F 3 "" H 1550 6950 60  0000 C CNN
-F 4 "digikey" H 1650 6700 60  0001 C CNN "Vendor"
-F 5 "102-1914-ND" H 1750 6800 60  0001 C CNN "PartNumber"
-F 6 "ENCODER OPT 32PPR DET CABLE TYPE" H 1850 6900 60  0001 C CNN "Description"
-	1    1550 6950
-	1    0    0    -1
-$EndComp
 $Comp
 L PWR_JACK_2.5x5.5 P1
@@
 	1    0    0    -1
 $EndComp
+$Comp
+L ENCODER_C14 E1
+U 1 1 548B59E0
+P 1550 6950
+F 0 "E1" H 1550 6600 60  0000 C CNN
+F 1 "ENCODER_C14" H 1550 7300 60  0000 C CNN
+F 2 "aalborg_mfc_interface:Micro-MaTch_6_SMD" H 1450 6500 60  0001 C CNN
+F 3 "" H 1550 6950 60  0000 C CNN
+F 4 "digikey" H 1650 6700 60  0001 C CNN "Vendor"
+F 5 "A99474CT-ND" H 1750 6800 60  0001 C CNN "PartNumber"
+F 6 "CONN FMALE-ON-BRD 6POS VERT SMD" H 1850 6900 60  0001 C CNN "Description"
+	1    1550 6950
+	1    0    0    -1
+$EndComp
